File: pcb/power_supply.kicad_sch (KiCad schematic)
At the start: 1 part, among them U2 BD9C301FJ

Commit message: Checkpoint
Parts:
- added C1, C2, C6: 47u, symbol Device:C_Polarized_Small_US
- added C3, C5: 100n, symbol Device:C_Small
- added C4: 10u, symbol Device:C_Small
- added C7, C8: 22u, symbol Device:C_Small
- added C9: 22n, symbol Device:C_Small
- added J2: USB_C_Receptacle_USB2.0_14P, symbol Connector:USB_C_Receptacle_USB2.0_14P
- added L1: 4.7u, symbol Device:L_Ferrite_Small
- added R1, R2: 5.1k, Resistor_SMD:R_0805_2012Metric, symbol Device:R_Small_US
- added R3: 2.4k, Resistor_SMD:R_0805_2012Metric, symbol Device:R_Small_US
- added R4: 7.5k, Resistor_SMD:R_0805_2012Metric, symbol Device:R_Small_US
- added R5: 12k, Resistor_SMD:R_0805_2012Metric, symbol Device:R_Small_US
- added U3: USBLC6-2SC6, Package_TO_SOT_SMD:SOT-23-6, symbol Power_Protection:USBLC6-2SC6
Connections:
- net GND: now reaches U2.1 (PGND)
- net GND: now also U2.3 (AGND), C1.2, C2.2, C3.2, C4.2, C5.2, C7.2, C8.2, C9.2, J2.A1 (GND), J2.A12 (GND), J2.B1 (GND), J2.B12 (GND), J2.S1 (SHIELD), R1.2, R2.2, R3.1, U3.2 (GND)
- net 5V_USB_SUP: now reaches U2.2 (VIN)
- net 5V_USB_SUP: now also C1.1, C2.1, C3.1, C4.1, C5.1, J2.A4 (VBUS), J2.A9 (VBUS), J2.B4 (VBUS), J2.B9 (VBUS), U3.5 (VBUS)
- net at U2.4 (FB): now also R3.2, R4.1
- net at U2.5 (COMP): now also R5.2
- net 3v3_BUCK_EN: now reaches U2.6 (EN)
- net at U2.7 (SW): now also U2.8 (SW), L1.1
- new net: J2.A6 (D+), J2.B6 (D+), U3.3 (I/O2)
- new net: J2.A7 (D-), J2.B7 (D-), U3.1 (I/O1)
- new net: C9.1, R5.1
- new net 3V3_SUP: C7.1, C8.1, L1.2, R4.2
- new net CC1: J2.A5 (CC1), R1.1
- new net CC2: J2.B5 (CC2), R2.1
- new net USB_D+: U3.4 (I/O2)
- new net USB_D-: U3.6 (I/O1)
Other:
- note added: "12.3kR Rcomp 23.6nF Ccomp @ 3.3V, 500mA, 44uF Cout"
- moved on the sheet: U2

Commit message: Checkpoint
Parts:
- added C10, C11, C12: 22u, symbol Device:C_Small
- added C13, C14: 4.7u, symbol Device:C_Small
- added D1: D_Schottky_Small, symbol Device:D_Schottky_Small
- added L2: 4.7u, symbol Device:L_Ferrite_Small
- added R6: 5.11, Resistor_SMD:R_0805_2012Metric, symbol Device:R_Small_US
- added U5: TPS61169, Package_TO_SOT_SMD:Texas_R-PDSO-G5_DCK-5, symbol custom-symbols:TPS61169
Connections:
- net 3V3_SUP: now also C10.1, C11.1, C12.1
- net 5V_USB_SUP: now also C13.1, L2.1, U5.5 (VIN)
- net GND: now also C10.2, C11.2, C12.2, C13.2, C14.2, R6.1, U5.2 (GND)
- new net: D1.2 (A), L2.2, U5.1 (SW)
- new net BKLGHT_A: C14.1, D1.1 (K)
- new net BKLGHT_K: R6.2, U5.3 (FB)
- new net BKLGHT_PWM: U5.4 (CTRL)
Other:
- note added: "Placement forseen but not required"
- moved on the sheet: C6, C7
