File: pcb/mcu_lcd.kicad_sch (KiCad schematic)
At the start: 2 parts, among them J1 Conn_01x40_Socket, U1 STM32H7B3IITx

Commit message: Checkpoint
Parts:
- added U4: XPT2046TS, Package_SO:TSSOP-16_4.4x5mm_P0.65mm, symbol Driver_Display:XPT2046TS
Changed lines of the file:
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@@
+	)
+	(symbol
+		(lib_id "Driver_Display:XPT2046TS")
+		(at 311.15 184.15 0)
+		(mirror y)
+		(unit 1)
+		(exclude_from_sim no)
+		(in_bom yes)
+		(on_board yes)
+		(dnp no)
+		(property "Reference" "U4"
+			(at 309.0067 196.85 0)
+			(effects
+				(font
+					(size 1.27 1.27)
+				)
+				(justify left)
+			)
+		)
+		(property "Value" "XPT2046TS"
+			(at 309.0067 199.39 0)
+			(effects
+				(font
+					(size 1.27 1.27)
+				)
+				(justify left)
+			)
+		)
+		(property "Footprint" "Package_SO:TSSOP-16_4.4x5mm_P0.65mm"
+			(at 311.15 199.39 0)
+			(effects
+				(font
+					(size 1.27 1.27)
+					(italic yes)
+				)
+				(hide yes)
+			)
+		)
+		(property "Datasheet" "http://www.xptek.cn/uploadfile/download/201707171401161883.pdf"
+			(at 306.07 198.12 0)
+			(effects
+				(font
+					(size 1.27 1.27)
+				)
+				(hide yes)
+			)
+		)
+		(property "Description" "Single-supply, 12bit, 4 ch, touch screen driver, 2.2 - 5.25 VDD, -40 to +85 C, QSPI, SPI, 3-wire serial interface, TSSOP-16"
+			(at 311.15 184.15 0)
+			(effects
+				(font
+					(size 1.27 1.27)
+				)
+				(hide yes)
+			)
+		)
+		(pin "4"
+		)
+		(pin "13"
+		)
+		(pin "11"
+		)
+		(pin "6"
+		)
+		(pin "2"
+		)
+		(pin "3"
+		)
+		(pin "8"
+		)
+		(pin "9"
+		)
+		(pin "7"
+		)
+		(pin "5"
+		)
+		(pin "16"
+		)
+		(pin "10"
+		)
+		(pin "1"
+		)
+		(pin "12"
+		)
+		(pin "15"
+		)
+		(pin "14"
+		)
+		(instances
+			(project ""
+				(path "/62b60f62-2f94-4785-a386-1becb3f82c7d/ab4c7c7d-a171-4841-b63a-3f82cac3161c"
+					(reference "U4")
+					(unit 1)
+				)
+			)
+		)
 	)
 	(symbol

Commit message: Checkpoint
Parts:
- added C18, C19, C20, C21, C22, C23, C24, C25, C26, C27, C28, C29, C30, C32: 100n, symbol Device:C_Small
- added C31: 10u, symbol Device:C_Small
- added R7: 10k, Resistor_SMD:R_0805_2012Metric, symbol Device:R_Small_US
- added SW1: SW_SPDT, symbol Switch:SW_SPDT
Connections:
- net GND: now reaches U1.102 (VSS), U1.113 (VSS), U1.126 (VSS), U1.135 (VSS), U1.14 (VSS), U1.148 (VSS), U1.158 (VSS), U1.22 (VSS), U1.48 (VSS), U1.61 (VSS), U1.71 (VSS), U1.90 (VSS)
- net GND: now also U1.37 (VSSA), C18.2, C19.2, C20.2, C21.2, C22.2, C23.2, C24.2, C25.2, C26.2, C27.2, C28.2, C29.2, C30.2, C31.2, C32.2, SW1.1 (A)
- net 3V3_SUP: now reaches U1.103 (VDD)
- net 3V3_SUP: now also U1.127 (VDD), U1.136 (VDD), U1.15 (VDD), U1.159 (VDD), U1.172 (VDD), U1.23 (VDD), U1.36 (VDD), U1.49 (VDD), U1.6 (VBAT), U1.62 (VDD), U1.72 (VDD), U1.82 (VDD), U1.91 (VDD), C18.1, C19.1, C20.1, C21.1, C22.1, C23.1, C24.1, C25.1, C26.1, C27.1, C28.1, C29.1, C30.1, C31.1, SW1.3 (C)
- net LTDC_VSYNC: now reaches U1.11 (PI9)
- net ADC1_INP7: now reaches U1.119 (PA8)
- net LTDC_HSYNC: now reaches U1.12 (PI10)
- net 5V_USB_SUP: now reaches U1.120 (PA9)
- net USB_OTG_HS_D-: now reaches U1.122 (PA11)
- net USB_OTG_HS_D+: now reaches U1.123 (PA12)
- net DEBUG_JTMS-SWDIO: now reaches U1.124 (PA13)
- net FDCAN1_TX: now reaches U1.128 (PH13)
- net FDCAN1_RX: now reaches U1.129 (PH14)
- net LTDC_G6: now reaches U1.13 (PI11)
- net DEBUG_JTCK-SWCLK: now reaches U1.137 (PA14)
- net LTDC_G7: now reaches U1.145 (PD3)
- net LTDC_B2: now reaches U1.150 (PD6)
- net LTDC_G3: now reaches U1.153 (PG10)
- net LTDC_B3: now reaches U1.154 (PG11)
- net LTDC_B1: now reaches U1.155 (PG12)
- net LTDC_B0: now reaches U1.157 (PG14)
- net DEBUG_JTDO-SWO: now reaches U1.161 (PB3)
- net I2S1_SDI: now reaches U1.162 (PB4)
- net I2S1_SDO: now reaches U1.163 (PB5)
- net BOOT0: now reaches U1.166 (BOOT0)
- net BOOT0: now also R7.2
- net LTDC_B4: now reaches U1.173 (PI4)
- net LTDC_B5: now reaches U1.174 (PI5)
- net LTDC_B6: now reaches U1.175 (PI6)
- net LTDC_B7: now reaches U1.176 (PI7)
- net LTDC_DE: now reaches U1.28 (PF10)
- net RCC_OSC_IN: now reaches U1.29 (PH0)
- net RCC_OSC_OUT: now reaches U1.30 (PH1)
- net NRST: now reaches U1.31 (NRST)
- net NRST: now also C32.1
- net LTDC_G2: now reaches U1.32 (PC0)
- net LTDC_G0: now reaches U1.4 (PE5)
- net LTDC_R0: now reaches U1.43 (PH2)
- net LTDC_R1: now reaches U1.44 (PH3)
- net LTDC_G1: now reaches U1.5 (PE6)
- net I2S1_WS: now reaches U1.50 (PA4)
- net I2S1_CLK: now reaches U1.51 (PA5)
- net ADC1_INP4: now reaches U1.54 (PC4)
- net ADC1_INP5: now reaches U1.57 (PB1)
- net ADC1_INP2: now reaches U1.59 (PF11)
- net ADC1_INP6: now reaches U1.60 (PF12)
- net LTDC_CLK: now reaches U1.77 (PE14)
- net LTDC_R7: now reaches U1.78 (PE15)
- net LTDC_G4: now reaches U1.79 (PB10)
- net LTDC_G5: now reaches U1.80 (PB11)
- net LTDC_R2: now reaches U1.85 (PH8)
- net LTDC_R3: now reaches U1.86 (PH9)
- net LTDC_R4: now reaches U1.87 (PH10)
- net LTDC_R5: now reaches U1.88 (PH11)
- net LTDC_R6: now reaches U1.89 (PH12)
- net SPI2_SCK: now reaches U1.93 (PB13)
- net SPI2_MISO: now reaches U1.94 (PB14)
- net SPI2_MOSI: now reaches U1.95 (PB15)
- new net: R7.1, SW1.2 (B)
Other:
- moved on the sheet: J1, U1, U4
